Commit message: -Change wry2 to be fixed (leads to atlas_v4 collapsing in drcsim 4.2 prerelease)

File: atlas_description/urdf/atlas_v4_simple_shapes.urdf (robot description, URDF)
Before this commit: robot drc_skeleton, 36 links, 36 joints
Joints:
- joint l_arm_wry2: type revolute -> fixed
- joint r_arm_wry2: type revolute -> fixed

Commit message: Pull in changes from drcsim_4.2 (no group names)

File: atlas_description/urdf/atlas_v4_simple_shapes.urdf (robot description, URDF)
Before this commit: robot drc_skeleton, 36 links, 36 joints
Links:
- link l_clav: geometry collision box size=0.1 0.07 0.072; collision cylinder length=0.1525 radius=0.0555
- link l_foot: geometry collision box size=${0.26-0.033} ${0.124887+0.009} 0.05; collision box size=0.1 ${0.08} 0.02
- link l_larm: geometry collision box size=0.135 0.15 0.06; collision cylinder length=0.125 radius=0.045
- link l_lfarm: geometry collision box size=0.13 0.09 0.07; collision cylinder length=0.05 radius=0.03
- link l_ufarm: geometry collision box size=0.135 0.1 0.045; collision cylinder length=0.125 radius=0.045
- link l_uleg: geometry collision box size=0.07 0.038 0.14; collision box size=0.07 0.038 0.15
- link r_clav: geometry collision box size=0.1 0.07 0.072; collision cylinder length=0.1525 radius=0.0555
- link r_foot: geometry collision box size=${0.26-0.033} ${0.124887+0.009} 0.05; collision box size=0.1 ${0.08} 0.02
- link r_larm: geometry collision box size=0.135 0.15 0.06; collision cylinder length=0.125 radius=0.045
- link r_lfarm: geometry collision box size=0.13 0.09 0.07; collision cylinder length=0.05 radius=0.03
- link r_ufarm: geometry collision box size=0.135 0.1 0.045; collision cylinder length=0.125 radius=0.045
- link r_uleg: geometry collision box size=0.07 0.038 0.14; collision box size=0.07 0.038 0.15
- link utorso: geometry collision box size=0.2 0.25 0.01; collision box size=0.456306 0.341719 0.12

File: atlas_description/urdf/atlas_v5_simple_shapes.urdf (robot description, URDF)
Before this commit: robot drc_skeleton, 36 links, 36 joints
Links:
- link l_foot: geometry collision box size=${0.26-0.033} ${0.124887+0.009} 0.05; collision box size=0.1 ${0.08} 0.02
- link r_foot: geometry collision box size=${0.26-0.033} ${0.124887+0.009} 0.05; collision box size=0.1 ${0.08} 0.02
