Commit message: Remove all use of wry2 joints

File: atlas_description/urdf/atlas_v4_no_wry2_simple_shapes.urdf (robot description, URDF)
Before this commit: robot drc_skeleton, 36 links, 36 joints
Joints:
- joint l_arm_wry2: axis 0 1 0 -> (none); limit lower=-0.001 upper=0.001 effort=5 velocity=1 -> (none); type revolute -> fixed
- joint r_arm_wry2: axis 0 1 0 -> (none); limit lower=-0.001 upper=0.001 effort=5 velocity=1 -> (none); type revolute -> fixed

Commit message: Remove wry2 joints and associated lfarm links, move lfarm geometry to hand links

File: atlas_description/urdf/atlas_v4_no_wry2_simple_shapes.urdf (robot description, URDF)
Before this commit: robot drc_skeleton, 36 links, 36 joints
Links:
- removed link l_lfarm
- removed link r_lfarm
- link l_hand: mass 0.1 -> 2.509; geometry collision box size=0.14 0.09 0.06; collision cylinder length=0.012 radius=0.048
- link r_hand: mass 0.1 -> 2.509; geometry collision box size=0.14 0.09 0.06; collision cylinder length=0.012 radius=0.048
Joints:
- removed joint l_arm_wry2
- removed joint r_arm_wry2
- joint l_arm_wrx: child l_lfarm -> l_hand
- joint r_arm_wrx: child r_lfarm -> r_hand

Commit message: Update collision geoms based on drcsim updates

File: atlas_description/urdf/atlas_v4_no_wry2_simple_shapes.urdf (robot description, URDF)
Before this commit: robot drc_skeleton, 34 links, 34 joints
Links:
- link l_clav: geometry collision box size=0.1 0.07 0.072; collision cylinder length=0.1525 radius=0.0555
- link l_foot: geometry collision box size=${0.26-0.033} ${0.124887+0.009} 0.05; collision box size=0.1 ${0.08} 0.02
- link l_hand: geometry collision box size=0.13 0.09 0.07; collision cylinder length=0.05 radius=0.03
- link l_larm: geometry collision box size=0.135 0.15 0.06; collision cylinder length=0.125 radius=0.045
- link l_ufarm: geometry collision box size=0.135 0.1 0.045; collision cylinder length=0.125 radius=0.045
- link l_uleg: geometry collision box size=0.07 0.038 0.14; collision box size=0.07 0.038 0.15
- link r_clav: geometry collision box size=0.1 0.07 0.072; collision cylinder length=0.1525 radius=0.0555
- link r_foot: geometry collision box size=${0.26-0.033} ${0.124887+0.009} 0.05; collision box size=0.1 ${0.08} 0.02
- link r_hand: geometry collision box size=0.13 0.09 0.07; collision cylinder length=0.05 radius=0.03
- link r_larm: geometry collision box size=0.135 0.15 0.06; collision cylinder length=0.125 radius=0.045
- link r_ufarm: geometry collision box size=0.135 0.1 0.045; collision cylinder length=0.125 radius=0.045
- link r_uleg: geometry collision box size=0.07 0.038 0.14; collision box size=0.07 0.038 0.15
- link utorso: geometry collision box size=0.2 0.25 0.01; collision box size=0.456306 0.341719 0.12

Commit message: Pull in changes from collision geom improvement PR on Bitbucket https://bitbucket.org/osrf/drcsim/pull-request/531

File: atlas_description/urdf/atlas_v4_no_wry2_simple_shapes.urdf (robot description, URDF)
Before this commit: robot drc_skeleton, 32 links, 32 joints
Links:
- link utorso: geometry collision box size=0.2 0.25 0.01; collision box size=0.500175 0.35 0.5

File: atlas_description/urdf/atlas_v4_simple_shapes.urdf (robot description, URDF)
Before this commit: robot drc_skeleton, 34 links, 34 joints
Links:
- link utorso: geometry collision box size=0.2 0.25 0.01; collision box size=0.500175 0.35 0.5

File: atlas_description/urdf/atlas_v5_simple_shapes.urdf (robot description, URDF)
Before this commit: robot drc_skeleton, 34 links, 34 joints
Links:
- link utorso: geometry collision box size=0.2 0.25 0.01; collision box size=0.500175 0.35 0.5
