Commit message: Add crash protection stl Add additional visual to utorso for crash protection

File: atlas_description/urdf/atlas_v5_simple_shapes.urdf (robot description, URDF)
Before this commit: robot drc_skeleton, 34 links, 34 joints
Links:
- link utorso: geometry collision box size=0.13 0.50 0.10; collision box size=0.2 0.18 0.10

Commit message: Fixed wry2 joint axis direction

File: atlas_description/urdf/atlas_v5_simple_shapes.urdf (robot description, URDF)
Before this commit: robot drc_skeleton, 34 links, 34 joints
Joints:
- joint l_arm_wry2: axis 0 1 0 -> 0 -1 0
