Commit message: Added includes for hand guard

File: atlas_description/robots/hands/l_robotiq_guard.urdf.xacro (robot description, xacro)
@@ -3,5 +3,5 @@
   <xacro:include filename="$(find flor_atlas_description)/robots/vigir_robotiq_guard.urdf.xacro" />
   <xacro:vigir_robotiq_guard prefix="left"  parent="l_hand">
-    <origin rpy="0 0 0" xyz="0 0.115 0.0"/>
+    <origin rpy="0 0 0" xyz="0 0.115 0.01"/>
   </xacro:vigir_robotiq_guard>
 </robot>

File: atlas_description/robots/hands/r_robotiq_guard.urdf.xacro (robot description, xacro)
@@ -3,5 +3,5 @@
   <xacro:include filename="$(find flor_atlas_description)/robots/vigir_robotiq_guard.urdf.xacro" />
   <xacro:vigir_robotiq_guard prefix="right" parent="r_hand">
-    <origin rpy="3.14159 3.14159 0" xyz="0 -0.115 0.0"/>
+    <origin rpy="3.14159 3.14159 0" xyz="0 -0.115 0.01"/>
   </xacro:vigir_robotiq_guard>
 </robot>

File: atlas_description/robots/vigir_atlas_v4_7dof.urdf.xacro (robot description, xacro)
@@ -6,4 +6,6 @@
 <!--  <xacro:include filename="$(find flor_atlas_description)/multisense/$(env FLOR_MULTISENSE_TYPE).urdf.xacro" />-->
   <xacro:include filename="$(find multisense_sl_description)/urdf/multisense_sl_v3.urdf" />
+  <xacro:include filename="$(find atlas_description)/robots/hands/$(env VIGIR_LEFT_GUARD_TYPE).urdf.xacro" />
+  <xacro:include filename="$(find atlas_description)/robots/hands/$(env VIGIR_RIGHT_GUARD_TYPE).urdf.xacro" />
   <xacro:include filename="$(find atlas_description)/robots/hands/$(env FLOR_LEFT_HAND_TYPE).urdf.xacro" />
   <xacro:include filename="$(find atlas_description)/robots/hands/$(env FLOR_RIGHT_HAND_TYPE).urdf.xacro" />
