Commit message: Changed path for robotiq urdf

File: atlas_description/robots/hands/l_robotiq.urdf.xacro (robot description, xacro)
@@ -1,18 +1,21 @@
 <?xml version="1.0" ?>
 <robot xmlns:xacro="http://playerstage.sourceforge.net/gazebo/xmlschema/#interface" name="l_robotiq" >
-<!--  <xacro:include filename="$(find flor_atlas_description)/robots/flor_robotiq_hand.urdf.xacro" />
+  <!--xacro:include filename="$(find robotiq_s_model_visualization)/cfg/s-model_mesh_macro.xacro" />
+  <xacro:s-model_mesh prefix="left_" parent="l_hand">
+    <origin rpy="3.14159 -1.57 3.14159" xyz="0 0.18 0.01"/>
+  </xacro:s-model_mesh-->
+  <!--xacro:include filename="$(find flor_atlas_description)/robots/flor_robotiq_hand.urdf.xacro" />
   <xacro:s-model_articulated prefix="left" parent="l_hand">
     <origin rpy="3.14159 -1.57 3.14159" xyz="0 0.18 0.01"/>
-  </xacro:s-model_articulated>-->
-  <xacro:include filename="$(find robotiq_hand_description)/urdf/robotiq_hand.urdf.xacro" />
+  </xacro:s-model_articulated-->
+  <xacro:include filename="$(find flor_robotiq_hands_tools)/urdf/robotiq_hand.urdf.xacro" />
   <!-- Set the initial hand position and orientation by changing 'rpy' and 'xyz'
   to mach the values in your actual robot. -->
-  <xacro:robotiq_hand prefix="l_" parent="l_hand" reflect="-1">
-    <origin rpy="3.14159 3.14159 3.14159" xyz="-0.00125 0.17 0.01"/>
+  <xacro:robotiq_hand prefix="left_" parent="l_hand" reflect="-1">
+    <origin rpy="3.14159 -1.57 3.14159" xyz="-0.00125 0.17 0.01"/>
   </xacro:robotiq_hand>
   <gazebo>
-    <!-- plugin for right RobotiQ hand -->
-    <plugin name="right_robotiq_hand_plugin" filename="libRobotiqHandPlugin.so">
-      <side>right</side>
+    <plugin name="left_robotiq_hand_plugin" filename="libRobotiqHandPlugin.so">
+      <side>left</side>
       <kp_position>5.0</kp_position>
       <kd_position>0.5</kd_position>

File: atlas_description/robots/hands/r_robotiq.urdf.xacro (robot description, xacro)
@@ -1,16 +1,19 @@
 <?xml version="1.0" ?>
 <robot xmlns:xacro="http://playerstage.sourceforge.net/gazebo/xmlschema/#interface" name="r_robotiq" >
-<!--  <xacro:include filename="$(find flor_atlas_description)/robots/flor_robotiq_hand.urdf.xacro" />
+  <!--xacro:include filename="$(find robotiq_s_model_visualization)/cfg/s-model_mesh_macro.xacro" />
+  <xacro:s-model_mesh prefix="right_" parent="r_hand">
+    <origin rpy="1.57 -1.57 0" xyz="0 -0.18 0.01"/>
+  </xacro:s-model_mesh-->
+  <!--xacro:include filename="$(find flor_atlas_description)/robots/flor_robotiq_hand.urdf.xacro" />
   <xacro:s-model_articulated prefix="right" parent="r_hand">
     <origin rpy="3.14159 -1.57 0" xyz="0 -0.18 0.01"/>
-  </xacro:s-model_articulated>-->
-  <xacro:include filename="$(find robotiq_hand_description)/urdf/robotiq_hand.urdf.xacro" />
+  </xacro:s-model_articulated-->
+  <xacro:include filename="$(find flor_robotiq_hands_tools)/urdf/robotiq_hand.urdf.xacro" />
   <!-- Set the initial hand position and orientation by changing 'rpy' and 'xyz'
   to mach the values in your actual robot. -->
-  <xacro:robotiq_hand prefix="r_" parent="r_hand" reflect="1">
-    <origin rpy="3.14159 0 0" xyz="-0.00125 -0.17 0.01"/>
+  <xacro:robotiq_hand prefix="right_" parent="r_hand" reflect="1">
+    <origin rpy="3.14159 -1.57 0" xyz="-0.00125 -0.17 0.01"/>
   </xacro:robotiq_hand>
   <gazebo>
-    <!-- plugin for right RobotiQ hand -->
     <plugin name="right_robotiq_hand_plugin" filename="libRobotiqHandPlugin.so">
       <side>right</side>

Commit message: Changed to call vigir robotiq urdf

File: atlas_description/robots/hands/l_robotiq.urdf.xacro (robot description, xacro)
@@ -1,18 +1,14 @@
 <?xml version="1.0" ?>
 <robot xmlns:xacro="http://playerstage.sourceforge.net/gazebo/xmlschema/#interface" name="l_robotiq" >
-  <!--xacro:include filename="$(find robotiq_s_model_visualization)/cfg/s-model_mesh_macro.xacro" />
-  <xacro:s-model_mesh prefix="left_" parent="l_hand">
-    <origin rpy="3.14159 -1.57 3.14159" xyz="0 0.18 0.01"/>
-  </xacro:s-model_mesh-->
-  <!--xacro:include filename="$(find flor_atlas_description)/robots/flor_robotiq_hand.urdf.xacro" />
+  <xacro:include filename="$(find flor_atlas_description)/robots/flor_robotiq_hand.urdf.xacro" />
   <xacro:s-model_articulated prefix="left" parent="l_hand">
     <origin rpy="3.14159 -1.57 3.14159" xyz="0 0.18 0.01"/>
-  </xacro:s-model_articulated-->
-  <xacro:include filename="$(find flor_robotiq_hands_tools)/urdf/robotiq_hand.urdf.xacro" />
+  </xacro:s-model_articulated>
   <!-- Set the initial hand position and orientation by changing 'rpy' and 'xyz'
-  to mach the values in your actual robot. -->
+  to mach the values in your actual robot.
+  <xacro:include filename="$(find robotiq_hand_description)/urdf/robotiq_hand.urdf.xacro" />
   <xacro:robotiq_hand prefix="left_" parent="l_hand" reflect="-1">
     <origin rpy="3.14159 -1.57 3.14159" xyz="-0.00125 0.17 0.01"/>
-  </xacro:robotiq_hand>
+  </xacro:robotiq_hand>-->
   <gazebo>
     <plugin name="left_robotiq_hand_plugin" filename="libRobotiqHandPlugin.so">

File: atlas_description/robots/hands/r_robotiq.urdf.xacro (robot description, xacro)
@@ -1,18 +1,14 @@
 <?xml version="1.0" ?>
 <robot xmlns:xacro="http://playerstage.sourceforge.net/gazebo/xmlschema/#interface" name="r_robotiq" >
-  <!--xacro:include filename="$(find robotiq_s_model_visualization)/cfg/s-model_mesh_macro.xacro" />
-  <xacro:s-model_mesh prefix="right_" parent="r_hand">
-    <origin rpy="1.57 -1.57 0" xyz="0 -0.18 0.01"/>
-  </xacro:s-model_mesh-->
-  <!--xacro:include filename="$(find flor_atlas_description)/robots/flor_robotiq_hand.urdf.xacro" />
+  <xacro:include filename="$(find flor_atlas_description)/robots/flor_robotiq_hand.urdf.xacro" />
   <xacro:s-model_articulated prefix="right" parent="r_hand">
     <origin rpy="3.14159 -1.57 0" xyz="0 -0.18 0.01"/>
-  </xacro:s-model_articulated-->
-  <xacro:include filename="$(find flor_robotiq_hands_tools)/urdf/robotiq_hand.urdf.xacro" />
+  </xacro:s-model_articulated>
   <!-- Set the initial hand position and orientation by changing 'rpy' and 'xyz'
-  to mach the values in your actual robot. -->
+  to mach the values in your actual robot.
+  <xacro:include filename="$(find robotiq_hand_description)/urdf/robotiq_hand.urdf.xacro" />
   <xacro:robotiq_hand prefix="right_" parent="r_hand" reflect="1">
     <origin rpy="3.14159 -1.57 0" xyz="-0.00125 -0.17 0.01"/>
-  </xacro:robotiq_hand>
+  </xacro:robotiq_hand>-->
   <gazebo>
     <plugin name="right_robotiq_hand_plugin" filename="libRobotiqHandPlugin.so">

Commit message: Simplified left hand rotation

File: atlas_description/robots/hands/l_robotiq.urdf.xacro (robot description, xacro)
@@ -3,5 +3,5 @@
   <xacro:include filename="$(find flor_atlas_description)/robots/flor_robotiq_hand.urdf.xacro" />
   <xacro:s-model_articulated prefix="left" parent="l_hand">
-    <origin rpy="3.14159 -1.57 3.14159" xyz="0 0.18 0.01"/>
+    <origin rpy="0 -1.57 0" xyz="0 0.18 0.01"/>
   </xacro:s-model_articulated>
   <!-- Set the initial hand position and orientation by changing 'rpy' and 'xyz'

Commit message: Changed robotiq hand transformation

File: atlas_description/robots/hands/l_robotiq.urdf.xacro (robot description, xacro)
@@ -3,5 +3,5 @@
   <xacro:include filename="$(find flor_atlas_description)/robots/flor_robotiq_hand.urdf.xacro" />
   <xacro:s-model_articulated prefix="left" parent="l_hand">
-    <origin rpy="0 -1.57 0" xyz="0 0.18 0.01"/>
+    <origin rpy="0 -1.57 0" xyz="0 0.23 0.0"/>
   </xacro:s-model_articulated>
   <!-- Set the initial hand position and orientation by changing 'rpy' and 'xyz'

File: atlas_description/robots/hands/r_robotiq.urdf.xacro (robot description, xacro)
@@ -3,5 +3,5 @@
   <xacro:include filename="$(find flor_atlas_description)/robots/flor_robotiq_hand.urdf.xacro" />
   <xacro:s-model_articulated prefix="right" parent="r_hand">
-    <origin rpy="3.14159 -1.57 0" xyz="0 -0.18 0.01"/>
+    <origin rpy="3.14159 -1.57 0" xyz="0 -0.23 0.0"/>
   </xacro:s-model_articulated>
   <!-- Set the initial hand position and orientation by changing 'rpy' and 'xyz'

Commit message: Changed use of guard env variable

File: atlas_description/robots/hands/l_robotiq.urdf.xacro (robot description, xacro)
@@ -2,6 +2,7 @@
 <robot xmlns:xacro="http://playerstage.sourceforge.net/gazebo/xmlschema/#interface" name="l_robotiq" >
   <xacro:include filename="$(find flor_atlas_description)/robots/flor_robotiq_hand.urdf.xacro" />
+  <xacro:include filename="$(find flor_atlas_description)/robots/$(optenv VIGIR_LEFT_GUARD_TYPE l_no_guard)_robotiq_hand_macros.urdf.xacro" />
   <xacro:s-model_articulated prefix="left" parent="l_hand">
-    <origin rpy="0 -1.57 0" xyz="0 0.18 0.01"/>
+    <origin rpy="0 -1.57 0" xyz="0 0.21 0.01"/>
   </xacro:s-model_articulated>
   <!-- Set the initial hand position and orientation by changing 'rpy' and 'xyz'

File: atlas_description/robots/hands/r_robotiq.urdf.xacro (robot description, xacro)
@@ -2,6 +2,7 @@
 <robot xmlns:xacro="http://playerstage.sourceforge.net/gazebo/xmlschema/#interface" name="r_robotiq" >
   <xacro:include filename="$(find flor_atlas_description)/robots/flor_robotiq_hand.urdf.xacro" />
+  <xacro:include filename="$(find flor_atlas_description)/robots/$(optenv VIGIR_RIGHT_GUARD_TYPE r_no_guard)_robotiq_hand_macros.urdf.xacro" />
   <xacro:s-model_articulated prefix="right" parent="r_hand">
-    <origin rpy="3.14159 -1.57 0" xyz="0 -0.18 0.01"/>
+    <origin rpy="3.14159 -1.57 0" xyz="0 -0.21 0.01"/>
   </xacro:s-model_articulated>
   <!-- Set the initial hand position and orientation by changing 'rpy' and 'xyz'

File: atlas_description/robots/vigir_atlas.urdf.xacro (robot description, xacro)
@@ -6,6 +6,4 @@
 <!--  <xacro:include filename="$(find flor_atlas_description)/multisense/$(env FLOR_MULTISENSE_TYPE).urdf.xacro" />-->
   <xacro:include filename="$(find multisense_sl_description)/urdf/multisense_sl_v3.urdf" />
-  <xacro:include filename="$(find atlas_description)/robots/hands/$(env VIGIR_LEFT_GUARD_TYPE).urdf.xacro" />
-  <xacro:include filename="$(find atlas_description)/robots/hands/$(env VIGIR_RIGHT_GUARD_TYPE).urdf.xacro" />
   <xacro:include filename="$(find atlas_description)/robots/hands/$(env FLOR_LEFT_HAND_TYPE).urdf.xacro" />
   <xacro:include filename="$(find atlas_description)/robots/hands/$(env FLOR_RIGHT_HAND_TYPE).urdf.xacro" />

File: atlas_description/robots/vigir_atlas_v4_7dof.urdf.xacro (robot description, xacro)
@@ -6,6 +6,4 @@
 <!--  <xacro:include filename="$(find flor_atlas_description)/multisense/$(env FLOR_MULTISENSE_TYPE).urdf.xacro" />-->
   <xacro:include filename="$(find multisense_sl_description)/urdf/multisense_sl_v3.urdf" />
-  <xacro:include filename="$(find atlas_description)/robots/hands/$(env VIGIR_LEFT_GUARD_TYPE).urdf.xacro" />
-  <xacro:include filename="$(find atlas_description)/robots/hands/$(env VIGIR_RIGHT_GUARD_TYPE).urdf.xacro" />
   <xacro:include filename="$(find atlas_description)/robots/hands/$(env FLOR_LEFT_HAND_TYPE).urdf.xacro" />
   <xacro:include filename="$(find atlas_description)/robots/hands/$(env FLOR_RIGHT_HAND_TYPE).urdf.xacro" />

Commit message: Updated robotiq transformation

File: atlas_description/robots/hands/l_robotiq.urdf.xacro (robot description, xacro)
@@ -4,5 +4,5 @@
   <xacro:include filename="$(find flor_atlas_description)/robots/$(optenv VIGIR_LEFT_GUARD_TYPE l_no_guard)_robotiq_hand_macros.urdf.xacro" />
   <xacro:s-model_articulated prefix="left" parent="l_hand">
-    <origin rpy="0 -1.57 0" xyz="0 0.23 0.0"/>
+    <origin rpy="0 -1.57 0" xyz="0 0.21 0.0"/>
   </xacro:s-model_articulated>
   <!-- Set the initial hand position and orientation by changing 'rpy' and 'xyz'

File: atlas_description/robots/hands/r_robotiq.urdf.xacro (robot description, xacro)
@@ -4,5 +4,5 @@
   <xacro:include filename="$(find flor_atlas_description)/robots/$(optenv VIGIR_RIGHT_GUARD_TYPE r_no_guard)_robotiq_hand_macros.urdf.xacro" />
   <xacro:s-model_articulated prefix="right" parent="r_hand">
-    <origin rpy="3.14159 -1.57 0" xyz="0 -0.23 0.0"/>
+    <origin rpy="3.14159 -1.57 0" xyz="0 -0.21 0.0"/>
   </xacro:s-model_articulated>
   <!-- Set the initial hand position and orientation by changing 'rpy' and 'xyz'

Commit message: Updated hand transform, rotation of 60 degrees to match real robot

File: atlas_description/robots/hands/l_robotiq.urdf.xacro (robot description, xacro)
@@ -4,5 +4,5 @@
   <xacro:include filename="$(find flor_atlas_description)/robots/$(optenv VIGIR_LEFT_GUARD_TYPE l_no_guard)_robotiq_hand_macros.urdf.xacro" />
   <xacro:s-model_articulated prefix="left" parent="l_hand">
-    <origin rpy="0 -1.57 0" xyz="0 0.21 0.01"/>
+    <origin rpy="0 1.047 0" xyz="0 0.21 0.01"/>
   </xacro:s-model_articulated>
   <!-- Set the initial hand position and orientation by changing 'rpy' and 'xyz'

File: atlas_description/robots/hands/r_robotiq.urdf.xacro (robot description, xacro)
@@ -4,5 +4,5 @@
   <xacro:include filename="$(find flor_atlas_description)/robots/$(optenv VIGIR_RIGHT_GUARD_TYPE r_no_guard)_robotiq_hand_macros.urdf.xacro" />
   <xacro:s-model_articulated prefix="right" parent="r_hand">
-    <origin rpy="3.14159 -1.57 0" xyz="0 -0.21 0.01"/>
+    <origin rpy="3.14159 1.047 0" xyz="0 -0.21 0.01"/>
   </xacro:s-model_articulated>
   <!-- Set the initial hand position and orientation by changing 'rpy' and 'xyz'

Commit message: Updated hand position

File: atlas_description/robots/hands/l_robotiq.urdf.xacro (robot description, xacro)
@@ -4,5 +4,5 @@
   <xacro:include filename="$(find flor_atlas_description)/robots/$(optenv VIGIR_LEFT_GUARD_TYPE l_no_guard)_robotiq_hand_macros.urdf.xacro" />
   <xacro:s-model_articulated prefix="left" parent="l_hand">
-    <origin rpy="0 1.047 0" xyz="0 0.21 0.01"/>
+    <origin rpy="0 -0.523 0" xyz="0 0.189 0.01"/>
   </xacro:s-model_articulated>
   <!-- Set the initial hand position and orientation by changing 'rpy' and 'xyz'

File: atlas_description/robots/hands/r_robotiq.urdf.xacro (robot description, xacro)
@@ -4,5 +4,5 @@
   <xacro:include filename="$(find flor_atlas_description)/robots/$(optenv VIGIR_RIGHT_GUARD_TYPE r_no_guard)_robotiq_hand_macros.urdf.xacro" />
   <xacro:s-model_articulated prefix="right" parent="r_hand">
-    <origin rpy="3.14159 1.047 0" xyz="0 -0.21 0.01"/>
+    <origin rpy="3.14159 -0.523 0" xyz="0 -0.189 0.01"/>
   </xacro:s-model_articulated>
   <!-- Set the initial hand position and orientation by changing 'rpy' and 'xyz'

Commit message: Updated hand position

File: atlas_description/robots/hands/l_robotiq.urdf.xacro (robot description, xacro)
@@ -4,5 +4,5 @@
   <xacro:include filename="$(find flor_atlas_description)/robots/$(optenv VIGIR_LEFT_GUARD_TYPE l_no_guard)_robotiq_hand_macros.urdf.xacro" />
   <xacro:s-model_articulated prefix="left" parent="l_hand">
-    <origin rpy="0 -1.57 0" xyz="0 0.21 0.0"/>
+    <origin rpy="0 -1.57 0" xyz="0 0.18 0.0"/>
   </xacro:s-model_articulated>
   <!-- Set the initial hand position and orientation by changing 'rpy' and 'xyz'

File: atlas_description/robots/hands/r_robotiq.urdf.xacro (robot description, xacro)
@@ -4,5 +4,5 @@
   <xacro:include filename="$(find flor_atlas_description)/robots/$(optenv VIGIR_RIGHT_GUARD_TYPE r_no_guard)_robotiq_hand_macros.urdf.xacro" />
   <xacro:s-model_articulated prefix="right" parent="r_hand">
-    <origin rpy="3.14159 -1.57 0" xyz="0 -0.21 0.0"/>
+    <origin rpy="3.14159 -1.57 0" xyz="0 -0.18 0.0"/>
   </xacro:s-model_articulated>
   <!-- Set the initial hand position and orientation by changing 'rpy' and 'xyz'

Commit message: Fixed left hand rotation

File: atlas_description/robots/hands/l_robotiq.urdf.xacro (robot description, xacro)
@@ -5,5 +5,5 @@
   <xacro:include filename="$(find flor_atlas_description)/robots/vigir_robotiq_palm_camera.urdf.xacro" />
   <xacro:s-model_articulated prefix="left" parent="l_hand">
-    <origin rpy="0 -1.57 0" xyz="0 0.18 0.0"/>
+    <origin rpy="0 -1.57 3.14159" xyz="0 -0.18 0.0"/>
   </xacro:s-model_articulated>
   <xacro:palm_camera prefix="left" />

Commit message: Modified hand pose in URDF

File: atlas_description/robots/hands/l_robotiq.urdf.xacro (robot description, xacro)
@@ -5,5 +5,5 @@
   <xacro:include filename="$(find flor_atlas_description)/robots/vigir_robotiq_palm_camera.urdf.xacro" />
   <xacro:s-model_articulated prefix="left" parent="l_hand">
-    <origin rpy="0 -1.57 0" xyz="0 0.18 0.0"/>
+    <origin rpy="0 -1.57 0" xyz="0 0.185 0.0"/>
   </xacro:s-model_articulated>
   <xacro:palm_camera prefix="left" />

File: atlas_description/robots/hands/r_robotiq.urdf.xacro (robot description, xacro)
@@ -5,5 +5,5 @@
   <xacro:include filename="$(find flor_atlas_description)/robots/vigir_robotiq_palm_camera.urdf.xacro" />
   <xacro:s-model_articulated prefix="right" parent="r_hand">
-    <origin rpy="3.14159 -1.57 0" xyz="0 -0.18 0.0"/>
+    <origin rpy="3.14159 -1.57 0" xyz="0 -0.185 0.0"/>
   </xacro:s-model_articulated>
   <xacro:palm_camera prefix="right" />

Commit message: Modified hand pose (again) in URDF

File: atlas_description/robots/hands/l_robotiq.urdf.xacro (robot description, xacro)
@@ -5,5 +5,5 @@
   <xacro:include filename="$(find flor_atlas_description)/robots/vigir_robotiq_palm_camera.urdf.xacro" />
   <xacro:s-model_articulated prefix="left" parent="l_hand">
-    <origin rpy="0 -1.57 0" xyz="0 0.185 0.0"/>
+    <origin rpy="0 -1.57 0" xyz="0 0.175 0.0"/>
   </xacro:s-model_articulated>
   <xacro:palm_camera prefix="left" />

File: atlas_description/robots/hands/r_robotiq.urdf.xacro (robot description, xacro)
@@ -5,5 +5,5 @@
   <xacro:include filename="$(find flor_atlas_description)/robots/vigir_robotiq_palm_camera.urdf.xacro" />
   <xacro:s-model_articulated prefix="right" parent="r_hand">
-    <origin rpy="3.14159 -1.57 0" xyz="0 -0.185 0.0"/>
+    <origin rpy="3.14159 -1.57 0" xyz="0 -0.175 0.0"/>
   </xacro:s-model_articulated>
   <xacro:palm_camera prefix="right" />
