Commit message: Remove hand links

File: atlas_self_filter_description/urdf/atlas_v3_simple_shapes.urdf (robot description, URDF)
Before this commit: robot drc_skeleton, 34 links, 34 joints
Links:
- removed link l_hand
- removed link r_hand

File: atlas_self_filter_description/urdf/atlas_v4_no_wry2_simple_shapes.urdf (robot description, URDF)
Before this commit: robot drc_skeleton, 34 links, 34 joints
Links:
- removed link l_hand
- removed link r_hand

File: atlas_self_filter_description/urdf/atlas_v4_simple_shapes.urdf (robot description, URDF)
Before this commit: robot drc_skeleton, 34 links, 34 joints
Links:
- removed link l_hand
- removed link r_hand

File: atlas_self_filter_description/urdf/atlas_v5_simple_shapes.urdf (robot description, URDF)
Before this commit: robot drc_skeleton, 34 links, 34 joints
Links:
- removed link l_hand
- removed link r_hand
