Commit message: Add proper general hand filter shape

File: atlas_self_filter_description/urdf/hand_filter_shapes.urdf (robot description, URDF)
Before this commit: robot drc_skeleton, 2 links, 0 joints
Links:
- link l_hand: mass 0.5839 -> None; geometry collision cylinder length=0.3 radius=0.15
- link r_hand: mass 0.5839 -> None; geometry collision cylinder length=0.3 radius=0.15

Commit message: Make hand filter shapes a little larger based on testing

File: atlas_self_filter_description/urdf/hand_filter_shapes.urdf (robot description, URDF)
Before this commit: robot drc_skeleton, 2 links, 0 joints
Links:
- link l_hand: geometry collision cylinder length=0.4 radius=0.15
- link r_hand: geometry collision cylinder length=0.4 radius=0.15
