Commit message: Guard prototyping

File: atlas_description/robots/vigir_atlas.urdf.xacro (robot description, xacro)
@@ -8,4 +8,28 @@
   <xacro:include filename="$(find atlas_description)/robots/hands/$(env FLOR_LEFT_HAND_TYPE).urdf.xacro" />
   <xacro:include filename="$(find atlas_description)/robots/hands/$(env FLOR_RIGHT_HAND_TYPE).urdf.xacro" />
+    <joint name="l_guard_joint" type="fixed">
+      <origin xyz="0.0  0.06 0.0215" rpy="0 ${3.14159265} 0"/>
+      <parent link="l_hand"/>
+      <child link="l_guard_link"/>
+    </joint>
+    <link name="l_guard_link">
+      <inertial>
+        <origin xyz="0 0 0" />
+        <mass value="0.01" />
+        <inertia  ixx="0.00000001" ixy="0.0"  ixz="0.0"  iyy="0.00000001"  iyz="0.0"  izz="0.00000001" />
+      </inertial>
+      <visual>
+        <origin xyz="0 0 0" rpy="0 0 0"/>
+        <geometry>
+          <mesh filename="package://flor_atlas_description/meshes/hand_guard_axis_adjusted_2000_poly_repaired.stl"/>
+        </geometry>
+      </visual>
+      <collision>
+        <origin xyz="0 0 0" rpy="0 0 0"/>
+        <geometry>
+          <mesh filename="package://flor_atlas_description/meshes/hand_guard_axis_adjusted_2000_poly_repaired.stl"/>
+        </geometry>
+      </collision>
+    </link>
   <!--Optionally, add artag (see #2074) -->
   <!--

Commit message: Offset the hand guard properly (within 1 mm in all directions)

File: atlas_description/robots/vigir_atlas.urdf.xacro (robot description, xacro)
@@ -9,5 +9,5 @@
   <xacro:include filename="$(find atlas_description)/robots/hands/$(env FLOR_RIGHT_HAND_TYPE).urdf.xacro" />
     <joint name="l_guard_joint" type="fixed">
-      <origin xyz="0.0  0.06 0.0215" rpy="0 ${3.14159265} 0"/>
+      <origin xyz="-0.001  0.0942 0.010" rpy="0 0 0"/>
       <parent link="l_hand"/>
       <child link="l_guard_link"/>
@@ -22,5 +22,5 @@
         <origin xyz="0 0 0" rpy="0 0 0"/>
         <geometry>
-          <mesh filename="package://flor_atlas_description/meshes/hand_guard_axis_adjusted_2000_poly_repaired.stl"/>
+          <mesh filename="package://flor_atlas_description/meshes/hand_guard_reoriented_10_09_30.stl"/>
         </geometry>
       </visual>
@@ -28,5 +28,5 @@
         <origin xyz="0 0 0" rpy="0 0 0"/>
         <geometry>
-          <mesh filename="package://flor_atlas_description/meshes/hand_guard_axis_adjusted_2000_poly_repaired.stl"/>
+          <mesh filename="package://flor_atlas_description/meshes/hand_guard_reoriented_10_09_30.stl"/>
         </geometry>
       </collision>

Commit message: Changed mesh name and commented out env guard variable

File: atlas_description/robots/vigir_atlas.urdf.xacro (robot description, xacro)
@@ -6,6 +6,6 @@
 <!--  <xacro:include filename="$(find flor_atlas_description)/multisense/$(env FLOR_MULTISENSE_TYPE).urdf.xacro" />-->
   <xacro:include filename="$(find multisense_sl_description)/urdf/multisense_sl_v3.urdf" />
-  <xacro:include filename="$(find atlas_description)/robots/hands/$(env VIGIR_LEFT_GUARD_TYPE).urdf.xacro" />
-  <xacro:include filename="$(find atlas_description)/robots/hands/$(env VIGIR_RIGHT_GUARD_TYPE).urdf.xacro" />
+  <!--xacro:include filename="$(find atlas_description)/robots/hands/$(env VIGIR_LEFT_GUARD_TYPE).urdf.xacro" /-->
+  <!--xacro:include filename="$(find atlas_description)/robots/hands/$(env VIGIR_RIGHT_GUARD_TYPE).urdf.xacro" /-->
   <xacro:include filename="$(find atlas_description)/robots/hands/$(env FLOR_LEFT_HAND_TYPE).urdf.xacro" />
   <xacro:include filename="$(find atlas_description)/robots/hands/$(env FLOR_RIGHT_HAND_TYPE).urdf.xacro" />
@@ -24,5 +24,5 @@
         <origin xyz="0 0 0" rpy="0 0 0"/>
         <geometry>
-          <mesh filename="package://flor_atlas_description/meshes/hand_guard_reoriented_10_09_30.stl"/>
+          <mesh filename="package://flor_atlas_description/meshes/vigir_robotiq_guard.stl"/>
         </geometry>
       </visual>
@@ -30,5 +30,5 @@
         <origin xyz="0 0 0" rpy="0 0 0"/>
         <geometry>
-          <mesh filename="package://flor_atlas_description/meshes/hand_guard_reoriented_10_09_30.stl"/>
+          <mesh filename="package://flor_atlas_description/meshes/vigir_robotiq_guard.stl"/>
         </geometry>
       </collision>

Commit message: Add frame fixed wrt hokuyo rotation in rotation center

File: atlas_description/robots/vigir_atlas.urdf.xacro (robot description, xacro)
@@ -4,8 +4,15 @@
   <xacro:include filename="$(find atlas_description)/urdf/$(optenv FLOR_ROBOT_TYPE atlas_v4_no_wry2).gazebo" />
   <xacro:include filename="$(find atlas_description)/urdf/$(optenv FLOR_ROBOT_TYPE atlas_v4_no_wry2).transmission" />
-<!--  <xacro:include filename="$(find flor_atlas_description)/multisense/$(env FLOR_MULTISENSE_TYPE).urdf.xacro" />-->
   <xacro:include filename="$(find multisense_sl_description)/urdf/multisense_sl_v3.urdf" />
   <xacro:include filename="$(find atlas_description)/robots/hands/$(optenv FLOR_LEFT_HAND_TYPE l_stump).urdf.xacro" />
   <xacro:include filename="$(find atlas_description)/robots/hands/$(optenv FLOR_RIGHT_HAND_TYPE r_stump).urdf.xacro" />
+  <!--Add a frame for use with high fidelity LIDAR projection-->
+  <link name="hokuyo_spin_axis_frame"/>
+  <joint name="hokoyo_spin_axis_joint" type="fixed">
+    <axis xyz="0 1 0" />
+    <origin xyz="${-0.0446+0.03} 0 0.0880" rpy="0 0 0"/>
+    <parent link="head"/>
+    <child link="hokuyo_spin_axis_frame"/>
+  </joint>
   <!--Optionally, add artag (see #2074) -->
   <!--

Commit message: Updated the guard in simulation to the new guard for test sprint four. Still not on the right arm.

File: atlas_description/robots/vigir_atlas.urdf.xacro (robot description, xacro)
@@ -24,5 +24,5 @@
         <origin xyz="0 0 0" rpy="0 0 0"/>
         <geometry>
-          <mesh filename="package://flor_atlas_description/meshes/vigir_robotiq_guard.stl"/>
+          <mesh filename="package://atlas_description/meshes/vigir_robotiq_guard.stl"/>
         </geometry>
       </visual>
@@ -30,5 +30,5 @@
         <origin xyz="0 0 0" rpy="0 0 0"/>
         <geometry>
-          <mesh filename="package://flor_atlas_description/meshes/vigir_robotiq_guard.stl"/>
+          <mesh filename="package://atlas_description/meshes/vigir_robotiq_guard.stl"/>
         </geometry>
       </collision>

Commit message: Add special treatment for Multisense depending on if sim or real robot

File: atlas_description/robots/vigir_atlas.urdf.xacro (robot description, xacro)
@@ -4,5 +4,5 @@
   <xacro:include filename="$(find atlas_description)/urdf/$(optenv FLOR_ROBOT_TYPE atlas_v4_no_wry2).gazebo" />
   <xacro:include filename="$(find atlas_description)/urdf/$(optenv FLOR_ROBOT_TYPE atlas_v4_no_wry2).transmission" />
-  <xacro:include filename="$(find multisense_sl_description)/urdf/multisense_sl_v3.urdf" />
+  <xacro:include filename="$(find atlas_description)/robots/multisense/$(optenv FLOR_MULTISENSE_TYPE sim)_multisense.urdf.xacro" />
   <xacro:include filename="$(find atlas_description)/robots/hands/$(optenv FLOR_LEFT_HAND_TYPE l_stump).urdf.xacro" />
   <xacro:include filename="$(find atlas_description)/robots/hands/$(optenv FLOR_RIGHT_HAND_TYPE r_stump).urdf.xacro" />

File: multisense_description_cr/urdf/multisenseSL.urdf (robot description, URDF)
Before this commit: robot multisense, 16 links, 15 joints
Links:
- link head: geometry collision box size=0.1311 0.12 0.1791; visual mesh filename=package://multisense_description/meshes/head.dae

Commit message: Rotated guard for virginia testing

File: atlas_description/robots/vigir_atlas.urdf.xacro (robot description, xacro)
@@ -12,5 +12,5 @@
   <link name="hokuyo_spin_axis_frame"/>
     <joint name="l_guard_joint" type="fixed">
-      <origin xyz="-0.001  0.0942 0.010" rpy="0 0 0"/>
+      <origin xyz="-0.001  0.0942 0.010" rpy="0 3.14159 0"/>
       <parent link="l_hand"/>
       <child link="l_guard_link"/>

Commit message: Removed manual guard addition in vigir_atlas.xacro.urdf, handled by the hand xacro

File: atlas_description/robots/vigir_atlas.urdf.xacro (robot description, xacro)
@@ -9,28 +9,4 @@
   <!--Add a frame for use with high fidelity LIDAR projection-->
   <link name="hokuyo_spin_axis_frame"/>
-    <joint name="l_guard_joint" type="fixed">
-      <origin xyz="-0.001  0.0942 0.010" rpy="0 3.14159 0"/>
-      <parent link="l_hand"/>
-      <child link="l_guard_link"/>
-    </joint>
-    <link name="l_guard_link">
-      <inertial>
-        <origin xyz="0 0 0" />
-        <mass value="0.01" />
-        <inertia  ixx="0.00000001" ixy="0.0"  ixz="0.0"  iyy="0.00000001"  iyz="0.0"  izz="0.00000001" />
-      </inertial>
-      <visual>
-        <origin xyz="0 0 0" rpy="0 0 0"/>
-        <geometry>
-          <mesh filename="package://atlas_description/meshes/vigir_robotiq_guard.stl"/>
-        </geometry>
-      </visual>
-      <collision>
-        <origin xyz="0 0 0" rpy="0 0 0"/>
-        <geometry>
-          <mesh filename="package://atlas_description/meshes/vigir_robotiq_guard.stl"/>
-        </geometry>
-      </collision>
-    </link>
   <joint name="hokoyo_spin_axis_joint" type="fixed">
     <axis xyz="0 1 0" />

Commit message: Add poking stick visuals (collision geom off for the moment)

File: atlas_description/robots/vigir_atlas.urdf.xacro (robot description, xacro)
@@ -15,4 +15,11 @@
     <child link="hokuyo_spin_axis_frame"/>
   </joint>
+  <xacro:include filename="$(find atlas_description)/urdf/poking_stick.urdf.xacro.xml" />
+  <xacro:poking_stick_macro parent="utorso" prefix="left" length="0.15">
+    <origin xyz="0.35 0.1128 0.3805" rpy="0 0 0"/>
+  </xacro:poking_stick_macro>
+  <xacro:poking_stick_macro parent="utorso" prefix="right" length="0.15">
+    <origin xyz="0.35 -0.1128 0.3805" rpy="0 0 0"/>
+  </xacro:poking_stick_macro>
   <!--Optionally, add artag (see #2074) -->
   <!--
