Commit message: Modify CR URDF

File: multisense_description_cr/urdf/multisenseSL.urdf (robot description, URDF)
Before this commit: robot multisense, 17 links, 16 joints
Links:
- removed link head_root
Joints:
- removed joint head_root_joint
- joint accel_joint: parent head_root -> head
- joint gyro_joint: parent head_root -> head
- joint mag_joint: parent head_root -> head

Commit message: Changed continuous joints to fixed

File: multisense_description_cr/urdf/multisenseSL.urdf (robot description, URDF)
Before this commit: robot multisense, 16 links, 15 joints
Joints:
- joint left_camera_optical_joint: type continuous -> fixed
- joint spindle_joint: type continuous -> fixed

Commit message: Revert "Changed continuous joints to fixed"
This reverts commit c55db648ab2817f71aeedee7b09317781b425619.

File: multisense_description_cr/urdf/multisenseSL.urdf (robot description, URDF)
Before this commit: robot multisense, 16 links, 15 joints
Joints:
- joint left_camera_optical_joint: type fixed -> continuous
- joint spindle_joint: type fixed -> continuous
