Commit message: Add hook geom and use it

File: vigir_atlas_addons_description/robots/flor_hook_hand.urdf.xacro (robot description, xacro)
@@ -19,5 +19,5 @@
     <collision>
       <geometry>
-        <mesh filename="package://flor_atlas_description/meshes_hook/hook_convex.stl"/>
+        <mesh filename="package://vigir_atlas_addons_description/meshes/hook_convex.stl"/>
       </geometry>
       <origin rpy="0 0 0" xyz="0 0.0 -0.0"/>
@@ -25,5 +25,5 @@
     <visual>
       <geometry>
-        <mesh filename="package://flor_atlas_description/meshes_hook/hook_convex.stl"/>
+        <mesh filename="package://vigir_atlas_addons_description/meshes/hook_convex.stl"/>
       </geometry>
       <origin rpy="0 0 0" xyz="0 -0.0 -0.0"/>
