Commit message: Add hand guard geom and adjust macros

File: vigir_atlas_addons_description/robots/l_robotiq_guard_robotiq_hand_macros.urdf.xacro (robot description, xacro)
@@ -5,5 +5,5 @@
         <origin xyz="0 -0.115 0" rpy="0 -1.57 0"/>
         <geometry>
-            <mesh filename="package://flor_atlas_description/meshes/vigir_robotiq_guard.stl" />
+            <mesh filename="package://vigir_atlas_addons_description/meshes/vigir_robotiq_guard.stl" />
         </geometry>
         <material name="black">
@@ -14,5 +14,5 @@
         <origin xyz="0 -0.115 0" rpy="0 -1.57 0"/>
         <geometry>
-            <mesh filename="package://flor_atlas_description/meshes/vigir_robotiq_guard.stl" />
+            <mesh filename="package://vigir_atlas_addons_description/meshes/vigir_robotiq_guard.stl" />
         </geometry>
             <material name="yellow">
